File: LEARNSAT_PoBoI/TVS_Diodes.kicad_sch (KiCad schematic)
At the start: 4 parts

Commit message: added footprints
Parts:
- D1, D2, D6, D7: footprint ONSC-SOD-323-2-477-02_V -> Vault:ONSC-SOD-323-2-477-02_V
