File: LEARNSAT_PoBoI/WatchDog.kicad_sch (KiCad schematic)
At the start: 12 parts, among them SW1 B3U-1000P, SW2 B3U-1000P, U1 MAX6746KA29+T, U2 SN74AUP1G08QDCKRQ1, U3 MAX6746KA29+T, U4 SN74AUP1G08QDCKRQ1

Commit message: added footprints
Parts:
- C1, C3: footprint CAPC0603(1608)100_L -> Vault:CAPC0603(1608)100_L
- C2, C4: footprint CAPC0402(1005)60_L -> Vault:CAPC0402(1005)60_L
- R1, R2: footprint RESC0805(2012)_L -> Vault:RESC0805(2012)_L
- SW1, SW2: footprint OMRON-B3U-1000_V -> Vault:OMRON-B3U-1000_V
- U1, U3: footprint FP-K8-5-IPC_C -> Vault:FP-K8-5-IPC_C
- U2, U4: footprint DCK0005A_N -> Vault:DCK0005A_N
