File: LEARNSAT_PoBoI/3V3Secondary.kicad_sch (KiCad schematic)
At the start: 17 parts, among them Q1 SI7164DP-T1-GE3, Q4 SI5418DU-T1-GE3, U12 INA219AIDCNR, U15 LTC4231IUD-2#TRPBF

Commit message: added footprints
Parts:
- C24: footprint CAPC1608X90X35ML15T15 -> Vault:CAPC1608X90X35ML15T15
- C27: footprint CAPC1608X90X40LL10T20 -> Vault:CAPC1608X90X40LL10T20
- C29: footprint FP-C0805C-DN-IPC_A -> Vault:FP-C0805C-DN-IPC_A
- D22: footprint ONSC-SOD-323-2-477-02_V -> Vault:ONSC-SOD-323-2-477-02_V
- Q1: footprint Vishay_S17-0173-SINGLE_MFG -> Vault:Vishay_S17-0173-SINGLE_MFG
- Q4: footprint SI5418DU-T1-GE3-Footprint-1 -> Vault:SI5418DU-T1-GE3-Footprint-1
- R13, R14: footprint FP-CRCW1210-e3-IPC_C -> Vault:FP-CRCW1210-e3-IPC_C
- R19: footprint FP-CR0805-IPC_A -> Vault:FP-CR0805-IPC_A
- R20, R21: footprint RESC0402(1005)_L -> Vault:RESC0402(1005)_L
- R26: footprint FP-CSR1206-IPC_C -> Vault:FP-CSR1206-IPC_C
- R29: footprint RESC1005X40X25ML05T05 -> Vault:RESC1005X40X25ML05T05
- R31: footprint FP-ESR01-IPC_C -> Vault:FP-ESR01-IPC_C
- R33: footprint RESC1005X40X25NL05T10 -> Vault:RESC1005X40X25NL05T10
- U12: footprint FP-DCN0008A-IPC_A -> Vault:FP-DCN0008A-IPC_A
- U15: footprint FP-UD-12-05-08-1855-IPC_A -> Vault:FP-UD-12-05-08-1855-IPC_A
Changed lines of the file:
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@@
 			)
 		)
-		(property "Footprint" "FP-CR0805-IPC_A"
+		(property "Footprint" "Vault:FP-CR0805-IPC_A"
 			(at 76.2 139.7 0)
 			(hide yes)
@@
 			)
 		)
-		(property "Footprint" "SI5418DU-T1-GE3-Footprint-1"
+		(property "Footprint" "Vault:SI5418DU-T1-GE3-Footprint-1"
 			(at 162.56 111.76 0)
 			(hide yes)
@@
 			)
 		)
-		(property "Footprint" "FP-UD-12-05-08-1855-IPC_A"
+		(property "Footprint" "Vault:FP-UD-12-05-08-1855-IPC_A"
 			(at 96.52 134.62 0)
 			(hide yes)
@@
 			)
 		)
-		(property "Footprint" "FP-C0805C-DN-IPC_A"
+		(property "Footprint" "Vault:FP-C0805C-DN-IPC_A"
 			(at 137.16 154.94 0)
 			(hide yes)
@@
 		(in_pos_files yes)
 		(dnp no)
-		(property "Reference" "#PWR?"
+		(property "Reference" "#PWR069"
 			(at 139.7 78.74 0)
 			(hide yes)
@@
 			(project "LEARNSAT_POBOY_v3.2.0"
 				(path "/31302da5-a970-4b2b-aa05-afcd06cb9d09/a1860061-8193-4c1d-812f-13791385bd89"
-					(reference "#PWR?")
+					(reference "#PWR069")
 					(unit 1)
 				)
@@
 		(in_pos_files yes)
 		(dnp no)
-		(property "Reference" "#PWR?"
+		(property "Reference" "#PWR071"
 			(at 154.94 154.94 0)
 			(hide yes)
@@
 			(project "LEARNSAT_POBOY_v3.2.0"
 				(path "/31302da5-a970-4b2b-aa05-afcd06cb9d09/a1860061-8193-4c1d-812f-13791385bd89"
-					(reference "#PWR?")
+					(reference "#PWR071")
 					(unit 1)
 				)
@@
 			)
 		)
-		(property "Footprint" "RESC0402(1005)_L"
+		(property "Footprint" "Vault:RESC0402(1005)_L"
 			(at 78.74 93.98 0)
 			(hide yes)
@@
 			)
 		)
-		(property "Footprint" "FP-CSR1206-IPC_C"
+		(property "Footprint" "Vault:FP-CSR1206-IPC_C"
 			(at 60.96 109.22 0)
 			(hide yes)
@@
 		(in_pos_files yes)
 		(dnp no)
-		(property "Reference" "#PWR?"
+		(property "Reference" "#PWR068"
 			(at 129.54 78.74 0)
 			(hide yes)
@@
 			(project "LEARNSAT_POBOY_v3.2.0"
 				(path "/31302da5-a970-4b2b-aa05-afcd06cb9d09/a1860061-8193-4c1d-812f-13791385bd89"
-					(reference "#PWR?")
+					(reference "#PWR068")
 					(unit 1)
 				)
@@
 			)
 		)
-		(property "Footprint" "CAPC1608X90X40LL10T20"
+		(property "Footprint" "Vault:CAPC1608X90X40LL10T20"
 			(at 81.28 76.2 0)
 			(hide yes)
@@
 			)
 		)
-		(property "Footprint" "FP-CRCW1210-e3-IPC_C"
+		(property "Footprint" "Vault:FP-CRCW1210-e3-IPC_C"
 			(at 129.54 48.26 0)
 			(hide yes)
@@
 			)
 		)
-		(property "Footprint" "ONSC-SOD-323-2-477-02_V"
+		(property "Footprint" "Vault:ONSC-SOD-323-2-477-02_V"
 			(at 165.1 157.48 0)
 			(hide yes)
@@
 		(in_pos_files yes)
 		(dnp no)
-		(property "Reference" "#PWR?"
+		(property "Reference" "#PWR067"
 			(at 121.92 35.56 0)
 			(hide yes)
@@
 			(project "LEARNSAT_POBOY_v3.2.0"
 				(path "/31302da5-a970-4b2b-aa05-afcd06cb9d09/a1860061-8193-4c1d-812f-13791385bd89"
-					(reference "#PWR?")
+					(reference "#PWR067")
 					(unit 1)
 				)
@@
 			)
 		)
-		(property "Footprint" "RESC0402(1005)_L"
+		(property "Footprint" "Vault:RESC0402(1005)_L"
 			(at 60.96 93.98 0)
 			(hide yes)
@@
 			)
 		)
-		(property "Footprint" "RESC1005X40X25NL05T10"
+		(property "Footprint" "Vault:RESC1005X40X25NL05T10"
 			(at 76.2 175.26 0)
 			(hide yes)
@@
 		(in_pos_files yes)
 		(dnp no)
-		(property "Reference" "#PWR?"
+		(property "Reference" "#PWR072"
 			(at 162.56 167.64 0)
 			(hide yes)
@@
 			(project "LEARNSAT_POBOY_v3.2.0"
 				(path "/31302da5-a970-4b2b-aa05-afcd06cb9d09/a1860061-8193-4c1d-812f-13791385bd89"
-					(reference "#PWR?")
+					(reference "#PWR072")
 					(unit 1)
 				)
@@
 			)
 		)
-		(property "Footprint" "FP-CRCW1210-e3-IPC_C"
+		(property "Footprint" "Vault:FP-CRCW1210-e3-IPC_C"
 			(at 139.7 48.26 0)
 			(hide yes)
@@
 			)
 		)
-		(property "Footprint" "FP-DCN0008A-IPC_A"
+		(property "Footprint" "Vault:FP-DCN0008A-IPC_A"
 			(at 93.98 63.5 0)
 			(hide yes)
@@
 		(in_pos_files yes)
 		(dnp no)
-		(property "Reference" "#PWR?"
+		(property "Reference" "#PWR070"
 			(at 144.78 170.18 0)
 			(hide yes)
@@
 			(project "LEARNSAT_POBOY_v3.2.0"
 				(path "/31302da5-a970-4b2b-aa05-afcd06cb9d09/a1860061-8193-4c1d-812f-13791385bd89"
-					(reference "#PWR?")
+					(reference "#PWR070")
 					(unit 1)
 				)
@@
 			)
 		)
-		(property "Footprint" "Vishay_S17-0173-SINGLE_MFG"
+		(property "Footprint" "Vault:Vishay_S17-0173-SINGLE_MFG"
 			(at 121.92 127 0)
 			(hide yes)
@@
 			)
 		)
-		(property "Footprint" "FP-ESR01-IPC_C"
+		(property "Footprint" "Vault:FP-ESR01-IPC_C"
 			(at 76.2 193.04 0)
 			(hide yes)
@@
 			)
 		)
-		(property "Footprint" "RESC1005X40X25ML05T05"
+		(property "Footprint" "Vault:RESC1005X40X25ML05T05"
 			(at 76.2 157.48 0)
 			(hide yes)
@@
 			)
 		)
-		(property "Footprint" "CAPC1608X90X35ML15T15"
+		(property "Footprint" "Vault:CAPC1608X90X35ML15T15"
 			(at 109.22 43.18 0)
 			(hide yes)
