File: LEARNSAT_PoBoI/5V_Buck.kicad_sch (KiCad schematic)
At the start: 22 parts, among them U8 LT1616ES6#TRMPBF, U9 LT1616ES6#TRMPBF

Commit message: added footprints
Parts:
- C13, C16, C17, C20: footprint FP-C0603-CJ-MFG -> Vault:FP-C0603-CJ-MFG
- C14, C18: footprint FP-CL10-IPC_B -> Vault:FP-CL10-IPC_B
- C15, C19: footprint CAPC0603(1608)100_L -> Vault:CAPC0603(1608)100_L
- D13, D15, D16, D18: footprint FP-502-01-MFG -> Vault:FP-502-01-MFG
- D14, D17: footprint FP-425-04-MFG -> Vault:FP-425-04-MFG
- L3, L4: footprint FP-LQH43CN_03-MFG -> Vault:FP-LQH43CN_03-MFG
- R10, R8: footprint RESC1609X50X30NL8T20 -> Vault:RESC1609X50X30NL8T20
- R7, R9: footprint FP-CRCW0603-e3-IPC_C -> Vault:FP-CRCW0603-e3-IPC_C
- U8, U9: footprint LT-S6-6-SOT-23_M -> Vault:LT-S6-6-SOT-23_M
Changed lines of the file:
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@@
 			)
 		)
-		(property "Footprint" "RESC1609X50X30NL8T20"
+		(property "Footprint" "Vault:RESC1609X50X30NL8T20"
 			(at 134.62 91.44 0)
 			(hide yes)
@@
 			)
 		)
-		(property "Footprint" "FP-CL10-IPC_B"
+		(property "Footprint" "Vault:FP-CL10-IPC_B"
 			(at 58.42 154.94 0)
 			(hide yes)
@@
 			)
 		)
-		(property "Footprint" "FP-502-01-MFG"
+		(property "Footprint" "Vault:FP-502-01-MFG"
 			(at 160.02 134.62 0)
 			(hide yes)
@@
 			)
 		)
-		(property "Footprint" "FP-CRCW0603-e3-IPC_C"
+		(property "Footprint" "Vault:FP-CRCW0603-e3-IPC_C"
 			(at 134.62 76.2 0)
 			(hide yes)
@@
 		(in_pos_files yes)
 		(dnp no)
-		(property "Reference" "#PWR?"
+		(property "Reference" "#PWR0108"
 			(at 180.34 147.32 0)
 			(hide yes)
@@
 			(project "LEARNSAT_POBOY_v3.2.0"
 				(path "/31302da5-a970-4b2b-aa05-afcd06cb9d09/e23bbc96-0550-4d6b-8bf1-525b54cf76b2"
-					(reference "#PWR?")
+					(reference "#PWR0108")
 					(unit 1)
 				)
@@
 		(in_pos_files yes)
 		(dnp no)
-		(property "Reference" "#PWR?"
+		(property "Reference" "#PWR0107"
 			(at 172.72 68.58 0)
 			(hide yes)
@@
 			(project "LEARNSAT_POBOY_v3.2.0"
 				(path "/31302da5-a970-4b2b-aa05-afcd06cb9d09/e23bbc96-0550-4d6b-8bf1-525b54cf76b2"
-					(reference "#PWR?")
+					(reference "#PWR0107")
 					(unit 1)
 				)
@@
 			)
 		)
-		(property "Footprint" "FP-CRCW0603-e3-IPC_C"
+		(property "Footprint" "Vault:FP-CRCW0603-e3-IPC_C"
 			(at 134.62 157.48 0)
 			(hide yes)
@@
 			)
 		)
-		(property "Footprint" "FP-C0603-CJ-MFG"
+		(property "Footprint" "Vault:FP-C0603-CJ-MFG"
 			(at 180.34 137.16 0)
 			(hide yes)
@@
 		(in_pos_files yes)
 		(dnp no)
-		(property "Reference" "#PWR?"
+		(property "Reference" "#PWR099"
 			(at 81.28 99.06 0)
 			(hide yes)
@@
 			(project "LEARNSAT_POBOY_v3.2.0"
 				(path "/31302da5-a970-4b2b-aa05-afcd06cb9d09/e23bbc96-0550-4d6b-8bf1-525b54cf76b2"
-					(reference "#PWR?")
+					(reference "#PWR099")
 					(unit 1)
 				)
@@
 		(in_pos_files yes)
 		(dnp no)
-		(property "Reference" "#PWR?"
+		(property "Reference" "#PWR0103"
 			(at 134.62 99.06 0)
 			(hide yes)
@@
 			(project "LEARNSAT_POBOY_v3.2.0"
 				(path "/31302da5-a970-4b2b-aa05-afcd06cb9d09/e23bbc96-0550-4d6b-8bf1-525b54cf76b2"
-					(reference "#PWR?")
+					(reference "#PWR0103")
 					(unit 1)
 				)
@@
 			)
 		)
-		(property "Footprint" "FP-LQH43CN_03-MFG"
+		(property "Footprint" "Vault:FP-LQH43CN_03-MFG"
 			(at 116.84 134.62 0)
 			(hide yes)
@@
 		(in_pos_files yes)
 		(dnp no)
-		(property "Reference" "#PWR?"
+		(property "Reference" "#PWR0105"
 			(at 142.24 99.06 0)
 			(hide yes)
@@
 			(project "LEARNSAT_POBOY_v3.2.0"
 				(path "/31302da5-a970-4b2b-aa05-afcd06cb9d09/e23bbc96-0550-4d6b-8bf1-525b54cf76b2"
-					(reference "#PWR?")
+					(reference "#PWR0105")
 					(unit 1)
 				)
@@
 			)
 		)
-		(property "Footprint" "CAPC0603(1608)100_L"
+		(property "Footprint" "Vault:CAPC0603(1608)100_L"
 			(at 142.24 76.2 0)
 			(hide yes)
@@
 			)
 		)
-		(property "Footprint" "LT-S6-6-SOT-23_M"
+		(property "Footprint" "Vault:LT-S6-6-SOT-23_M"
 			(at 71.12 127 0)
 			(hide yes)
@@
 			)
 		)
-		(property "Footprint" "FP-C0603-CJ-MFG"
+		(property "Footprint" "Vault:FP-C0603-CJ-MFG"
 			(at 106.68 124.46 0)
 			(hide yes)
@@
 		(in_pos_files yes)
 		(dnp no)
-		(property "Reference" "#PWR?"
+		(property "Reference" "#PWR0106"
 			(at 147.32 180.34 0)
 			(hide yes)
@@
 			(project "LEARNSAT_POBOY_v3.2.0"
 				(path "/31302da5-a970-4b2b-aa05-afcd06cb9d09/e23bbc96-0550-4d6b-8bf1-525b54cf76b2"
-					(reference "#PWR?")
+					(reference "#PWR0106")
 					(unit 1)
 				)
@@
 			)
 		)
-		(property "Footprint" "FP-502-01-MFG"
+		(property "Footprint" "Vault:FP-502-01-MFG"
 			(at 129.54 38.1 0)
 			(hide yes)
@@
 		(in_pos_files yes)
 		(dnp no)
-		(property "Reference" "#PWR?"
+		(property "Reference" "#PWR098"
 			(at 58.42 180.34 0)
 			(hide yes)
@@
 			(project "LEARNSAT_POBOY_v3.2.0"
 				(path "/31302da5-a970-4b2b-aa05-afcd06cb9d09/e23bbc96-0550-4d6b-8bf1-525b54cf76b2"
-					(reference "#PWR?")
+					(reference "#PWR098")
 					(unit 1)
 				)
@@
 			)
 		)
-		(property "Footprint" "FP-C0603-CJ-MFG"
+		(property "Footprint" "Vault:FP-C0603-CJ-MFG"
 			(at 172.72 60.96 0)
 			(hide yes)
@@
 		(in_pos_files yes)
 		(dnp no)
-		(property "Reference" "#PWR?"
+		(property "Reference" "#PWR097"
 			(at 55.88 99.06 0)
 			(hide yes)
@@
 			(project "LEARNSAT_POBOY_v3.2.0"
 				(path "/31302da5-a970-4b2b-aa05-afcd06cb9d09/e23bbc96-0550-4d6b-8bf1-525b54cf76b2"
-					(reference "#PWR?")
+					(reference "#PWR097")
 					(unit 1)
 				)
@@
 			)
 		)
-		(property "Footprint" "FP-LQH43CN_03-MFG"
+		(property "Footprint" "Vault:FP-LQH43CN_03-MFG"
 			(at 116.84 53.34 0)
 			(hide yes)
@@
 		(in_pos_files yes)
 		(dnp no)
-		(property "Reference" "#PWR?"
+		(property "Reference" "#PWR0102"
 			(at 111.76 182.88 0)
 			(hide yes)
@@
 			(project "LEARNSAT_POBOY_v3.2.0"
 				(path "/31302da5-a970-4b2b-aa05-afcd06cb9d09/e23bbc96-0550-4d6b-8bf1-525b54cf76b2"
-					(reference "#PWR?")
+					(reference "#PWR0102")
 					(unit 1)
 				)
@@
 			)
 		)
-		(property "Footprint" "FP-CL10-IPC_B"
+		(property "Footprint" "Vault:FP-CL10-IPC_B"
 			(at 55.88 71.12 0)
 			(hide yes)
@@
 		(in_pos_files yes)
 		(dnp no)
-		(property "Reference" "#PWR?"
+		(property "Reference" "#PWR0101"
 			(at 111.76 99.06 0)
 			(hide yes)
@@
 			(project "LEARNSAT_POBOY_v3.2.0"
 				(path "/31302da5-a970-4b2b-aa05-afcd06cb9d09/e23bbc96-0550-4d6b-8bf1-525b54cf76b2"
-					(reference "#PWR?")
+					(reference "#PWR0101")
 					(unit 1)
 				)
@@
 			)
 		)
-		(property "Footprint" "FP-502-01-MFG"
+		(property "Footprint" "Vault:FP-502-01-MFG"
 			(at 152.4 55.88 0)
 			(hide yes)
@@
 		(in_pos_files yes)
 		(dnp no)
-		(property "Reference" "#PWR?"
+		(property "Reference" "#PWR0100"
 			(at 81.28 180.34 0)
 			(hide yes)
@@
 			(project "LEARNSAT_POBOY_v3.2.0"
 				(path "/31302da5-a970-4b2b-aa05-afcd06cb9d09/e23bbc96-0550-4d6b-8bf1-525b54cf76b2"
-					(reference "#PWR?")
+					(reference "#PWR0100")
 					(unit 1)
 				)
@@
 			)
 		)
-		(property "Footprint" "FP-502-01-MFG"
+		(property "Footprint" "Vault:FP-502-01-MFG"
 			(at 127 119.38 0)
 			(hide yes)
@@
 			)
 		)
-		(property "Footprint" "LT-S6-6-SOT-23_M"
+		(property "Footprint" "Vault:LT-S6-6-SOT-23_M"
 			(at 71.12 45.72 0)
 			(hide yes)
@@
 			)
 		)
-		(property "Footprint" "FP-C0603-CJ-MFG"
+		(property "Footprint" "Vault:FP-C0603-CJ-MFG"
 			(at 106.68 43.18 0)
 			(hide yes)
@@
 			)
 		)
-		(property "Footprint" "FP-425-04-MFG"
+		(property "Footprint" "Vault:FP-425-04-MFG"
 			(at 111.76 73.66 0)
 			(hide yes)
@@
 			)
 		)
-		(property "Footprint" "RESC1609X50X30NL8T20"
+		(property "Footprint" "Vault:RESC1609X50X30NL8T20"
 			(at 134.62 167.64 0)
 			(hide yes)
@@
 			)
 		)
-		(property "Footprint" "FP-425-04-MFG"
+		(property "Footprint" "Vault:FP-425-04-MFG"
 			(at 111.76 157.48 0)
 			(hide yes)
@@
 		(in_pos_files yes)
 		(dnp no)
-		(property "Reference" "#PWR?"
+		(property "Reference" "#PWR0104"
 			(at 134.62 180.34 0)
 			(hide yes)
@@
 			(project "LEARNSAT_POBOY_v3.2.0"
 				(path "/31302da5-a970-4b2b-aa05-afcd06cb9d09/e23bbc96-0550-4d6b-8bf1-525b54cf76b2"
-					(reference "#PWR?")
+					(reference "#PWR0104")
 					(unit 1)
 				)
@@
 			)
 		)
-		(property "Footprint" "CAPC0603(1608)100_L"
+		(property "Footprint" "Vault:CAPC0603(1608)100_L"
 			(at 147.32 149.86 0)
 			(hide yes)
