File: LEARNSAT_PoBoI/PC104.kicad_sch (KiCad schematic)
At the start: 28 parts, among them J1 FTSH-105-01-L-DV-K-P-TR, P1 22-28-4036, SW3 TS04-66-43-BK-100-SMT

Commit message: added footprints
Parts:
- 111: renamed from 1; footprint TP06R -> Vault:TP06R
- 211: renamed from 2; footprint TP06R -> Vault:TP06R
- 311: renamed from 3; footprint TP06R -> Vault:TP06R
- 411: renamed from 4; footprint TP06R -> Vault:TP06R
- 511: renamed from 5; footprint TP06R -> Vault:TP06R
- 611: renamed from 6; footprint TP06R -> Vault:TP06R
- C22: footprint FP-C0603-CJ-MFG -> Vault:FP-C0603-CJ-MFG
- GND1, VBATT1, VBATTP1, VBATTS1: footprint TP06R -> Vault:TP06R
- H1, H2: footprint SMTC-SSQ-126-22-X-D -> Vault:SMTC-SSQ-126-22-X-D
- J1: footprint FP-FTSH-105-01-L-DV-K-P-T-MFG -> Vault:FP-FTSH-105-01-L-DV-K-P-T-MFG
- LED1, LED2, LED3, LED4, LED5, LED6: footprint FP-HSMS-C150-MFG -> Vault:FP-HSMS-C150-MFG
- P1: footprint 22-28-4036-Footprint-1 -> Vault:22-28-4036-Footprint-1
- RLED1, RLED4: footprint FP-CRCW0603-e3-IPC_B -> Vault:FP-CRCW0603-e3-IPC_B
- RLED2, RLED5: footprint RESC1608X55X30NL20T20 -> Vault:RESC1608X55X30NL20T20
- RLED3, RLED6: footprint RESC1608X55X25ML10T15 -> Vault:RESC1608X55X25ML10T15
- SW3: footprint SOP127P600-8N -> Vault:SOP127P600-8N; DATASHEET https://www.cuidevices.com/product/resource/ts04.pdf -> (none)
