File: LEARNSAT_PoBoI/VBATTPrimary.kicad_sch (KiCad schematic)
At the start: 17 parts, among them Q12 SI7164DP-T1-GE3, Q13 SI5418DU-T1-GE3, U27 INA219AIDCNR, U29 LTC4231IUD-2#TRPBF

Commit message: minor naming changes
Parts:
- renumbered Q12 to Q14
Changed lines of the file:
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@@
 		(in_pos_files yes)
 		(dnp no)
-		(property "Reference" "#PWR?"
+		(property "Reference" "#PWR044"
 			(at 154.94 154.94 0)
 			(hide yes)
@@
 			(project "LEARNSAT_POBOY_v3.2.0"
 				(path "/31302da5-a970-4b2b-aa05-afcd06cb9d09/55f06696-b2d9-4c25-98ea-711c3045af0d"
-					(reference "#PWR?")
+					(reference "#PWR044")
 					(unit 1)
 				)
@@
 		(in_pos_files yes)
 		(dnp no)
-		(property "Reference" "#PWR?"
+		(property "Reference" "#PWR043"
 			(at 144.78 170.18 0)
 			(hide yes)
@@
 			(project "LEARNSAT_POBOY_v3.2.0"
 				(path "/31302da5-a970-4b2b-aa05-afcd06cb9d09/55f06696-b2d9-4c25-98ea-711c3045af0d"
-					(reference "#PWR?")
+					(reference "#PWR043")
 					(unit 1)
 				)
@@
 		(in_pos_files yes)
 		(dnp no)
-		(property "Reference" "#PWR?"
+		(property "Reference" "#PWR040"
 			(at 121.92 35.56 0)
 			(hide yes)
@@
 			(project "LEARNSAT_POBOY_v3.2.0"
 				(path "/31302da5-a970-4b2b-aa05-afcd06cb9d09/55f06696-b2d9-4c25-98ea-711c3045af0d"
-					(reference "#PWR?")
+					(reference "#PWR040")
 					(unit 1)
 				)
@@
 		(in_pos_files yes)
 		(dnp no)
-		(property "Reference" "Q12"
+		(property "Reference" "Q14"
 			(at 116.84 114.3 0)
 			(show_name no)
@@
 			(project "LEARNSAT_POBOY_v3.2.0"
 				(path "/31302da5-a970-4b2b-aa05-afcd06cb9d09/55f06696-b2d9-4c25-98ea-711c3045af0d"
-					(reference "Q12")
+					(reference "Q14")
 					(unit 1)
 				)
@@
 		(in_pos_files yes)
 		(dnp no)
-		(property "Reference" "#PWR?"
+		(property "Reference" "#PWR045"
 			(at 162.56 167.64 0)
 			(hide yes)
@@
 			(project "LEARNSAT_POBOY_v3.2.0"
 				(path "/31302da5-a970-4b2b-aa05-afcd06cb9d09/55f06696-b2d9-4c25-98ea-711c3045af0d"
-					(reference "#PWR?")
+					(reference "#PWR045")
 					(unit 1)
 				)
@@
 		(in_pos_files yes)
 		(dnp no)
-		(property "Reference" "#PWR?"
+		(property "Reference" "#PWR042"
 			(at 139.7 78.74 0)
 			(hide yes)
@@
 			(project "LEARNSAT_POBOY_v3.2.0"
 				(path "/31302da5-a970-4b2b-aa05-afcd06cb9d09/55f06696-b2d9-4c25-98ea-711c3045af0d"
-					(reference "#PWR?")
+					(reference "#PWR042")
 					(unit 1)
 				)
@@
 		(in_pos_files yes)
 		(dnp no)
-		(property "Reference" "#PWR?"
+		(property "Reference" "#PWR041"
 			(at 129.54 78.74 0)
 			(hide yes)
@@
 			(project "LEARNSAT_POBOY_v3.2.0"
 				(path "/31302da5-a970-4b2b-aa05-afcd06cb9d09/55f06696-b2d9-4c25-98ea-711c3045af0d"
-					(reference "#PWR?")
+					(reference "#PWR041")
 					(unit 1)
 				)
