File: LEARNSAT_PoBoI/5VSecondary.kicad_sch (KiCad schematic)
At the start: 17 parts, among them Q6 SI7164DP-T1-GE3, Q8 SI5418DU-T1-GE3, U19 INA219AIDCNR, U24 LTC4231IUD-2#TRPBF

Commit message: retried naming changes
Parts:
- C36: footprint CAPC1608X90X35ML15T15 -> Vault:CAPC1608X90X35ML15T15
- C37: footprint CAPC1608X90X40LL10T20 -> Vault:CAPC1608X90X40LL10T20
- C41: footprint FP-C0805C-DN-IPC_A -> Vault:FP-C0805C-DN-IPC_A
- D27: renamed from D23; footprint ONSC-SOD-323-2-477-02_V -> Vault:ONSC-SOD-323-2-477-02_V
- Q6: footprint Vishay_S17-0173-SINGLE_MFG -> Vault:Vishay_S17-0173-SINGLE_MFG
- Q8: footprint SI5418DU-T1-GE3-Footprint-1 -> Vault:SI5418DU-T1-GE3-Footprint-1
- R41, R42: footprint FP-CRCW1210-e3-IPC_C -> Vault:FP-CRCW1210-e3-IPC_C
- R45, R46, R52: footprint RESC0402(1005)_L -> Vault:RESC0402(1005)_L
- R47: footprint FP-CSR1206-IPC_C -> Vault:FP-CSR1206-IPC_C
- R53: footprint FP-PTN0603-IPC_B -> Vault:FP-PTN0603-IPC_B
- R54: footprint FP-CRCW1206-e3-IPC_A -> Vault:FP-CRCW1206-e3-IPC_A
- R55: footprint FP-RT1206-IPC_C -> Vault:FP-RT1206-IPC_C
- U19: footprint FP-DCN0008A-IPC_A -> Vault:FP-DCN0008A-IPC_A
- U24: footprint FP-UD-12-05-08-1855-IPC_A -> Vault:FP-UD-12-05-08-1855-IPC_A
Changed lines of the file:
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@@
 		(in_pos_files yes)
 		(dnp no)
-		(property "Reference" "#PWR?"
+		(property "Reference" "#PWR093"
 			(at 139.7 78.74 0)
 			(hide yes)
@@
 			(project "LEARNSAT_POBOY_v3.2.0"
 				(path "/31302da5-a970-4b2b-aa05-afcd06cb9d09/7afe09a5-989f-4cf0-b7aa-6eaacc747d01"
-					(reference "#PWR?")
+					(reference "#PWR093")
 					(unit 1)
 				)
@@
 			)
 		)
-		(property "Footprint" "FP-CRCW1210-e3-IPC_C"
+		(property "Footprint" "Vault:FP-CRCW1210-e3-IPC_C"
 			(at 129.54 48.26 0)
 			(hide yes)
@@
 		(in_pos_files yes)
 		(dnp no)
-		(property "Reference" "#PWR?"
+		(property "Reference" "#PWR095"
 			(at 154.94 154.94 0)
 			(hide yes)
@@
 			(project "LEARNSAT_POBOY_v3.2.0"
 				(path "/31302da5-a970-4b2b-aa05-afcd06cb9d09/7afe09a5-989f-4cf0-b7aa-6eaacc747d01"
-					(reference "#PWR?")
+					(reference "#PWR095")
 					(unit 1)
 				)
@@
 		(in_pos_files yes)
 		(dnp no)
-		(property "Reference" "#PWR?"
+		(property "Reference" "#PWR091"
 			(at 121.92 35.56 0)
 			(hide yes)
@@
 			(project "LEARNSAT_POBOY_v3.2.0"
 				(path "/31302da5-a970-4b2b-aa05-afcd06cb9d09/7afe09a5-989f-4cf0-b7aa-6eaacc747d01"
-					(reference "#PWR?")
+					(reference "#PWR091")
 					(unit 1)
 				)
@@
 			)
 		)
-		(property "Footprint" "Vishay_S17-0173-SINGLE_MFG"
+		(property "Footprint" "Vault:Vishay_S17-0173-SINGLE_MFG"
 			(at 121.92 129.54 0)
 			(hide yes)
@@
 			)
 		)
-		(property "Footprint" "FP-CRCW1206-e3-IPC_A"
+		(property "Footprint" "Vault:FP-CRCW1206-e3-IPC_A"
 			(at 76.2 157.48 0)
 			(hide yes)
@@
 			)
 		)
-		(property "Footprint" "FP-RT1206-IPC_C"
+		(property "Footprint" "Vault:FP-RT1206-IPC_C"
 			(at 76.2 193.04 0)
 			(hide yes)
@@
 			)
 		)
-		(property "Footprint" "CAPC1608X90X35ML15T15"
+		(property "Footprint" "Vault:CAPC1608X90X35ML15T15"
 			(at 109.22 43.18 0)
 			(hide yes)
@@
 			)
 		)
-		(property "Footprint" "RESC0402(1005)_L"
+		(property "Footprint" "Vault:RESC0402(1005)_L"
 			(at 60.96 93.98 0)
 			(hide yes)
@@
 			)
 		)
-		(property "Footprint" "FP-UD-12-05-08-1855-IPC_A"
+		(property "Footprint" "Vault:FP-UD-12-05-08-1855-IPC_A"
 			(at 96.52 134.62 0)
 			(hide yes)
@@
 			)
 		)
-		(property "Footprint" "FP-CRCW1210-e3-IPC_C"
+		(property "Footprint" "Vault:FP-CRCW1210-e3-IPC_C"
 			(at 139.7 48.26 0)
 			(hide yes)
@@
 		(in_pos_files yes)
 		(dnp no)
-		(property "Reference" "#PWR?"
+		(property "Reference" "#PWR094"
 			(at 144.78 167.64 0)
 			(hide yes)
@@
 			(project "LEARNSAT_POBOY_v3.2.0"
 				(path "/31302da5-a970-4b2b-aa05-afcd06cb9d09/7afe09a5-989f-4cf0-b7aa-6eaacc747d01"
-					(reference "#PWR?")
+					(reference "#PWR094")
 					(unit 1)
 				)
@@
 		(in_pos_files yes)
 		(dnp no)
-		(property "Reference" "#PWR?"
+		(property "Reference" "#PWR096"
 			(at 162.56 167.64 0)
 			(hide yes)
@@
 			(project "LEARNSAT_POBOY_v3.2.0"
 				(path "/31302da5-a970-4b2b-aa05-afcd06cb9d09/7afe09a5-989f-4cf0-b7aa-6eaacc747d01"
-					(reference "#PWR?")
+					(reference "#PWR096")
 					(unit 1)
 				)
@@
 			)
 		)
-		(property "Footprint" "FP-DCN0008A-IPC_A"
+		(property "Footprint" "Vault:FP-DCN0008A-IPC_A"
 			(at 93.98 63.5 0)
 			(hide yes)
@@
 			)
 		)
-		(property "Footprint" "RESC0402(1005)_L"
+		(property "Footprint" "Vault:RESC0402(1005)_L"
 			(at 78.74 93.98 0)
 			(hide yes)
@@
 		(in_pos_files yes)
 		(dnp no)
-		(property "Reference" "D23"
+		(property "Reference" "D27"
 			(at 165.1 160.02 0)
 			(show_name no)
@@
 			)
 		)
-		(property "Footprint" "ONSC-SOD-323-2-477-02_V"
+		(property "Footprint" "Vault:ONSC-SOD-323-2-477-02_V"
 			(at 165.1 157.48 0)
 			(hide yes)
@@
 			(project "LEARNSAT_POBOY_v3.2.0"
 				(path "/31302da5-a970-4b2b-aa05-afcd06cb9d09/7afe09a5-989f-4cf0-b7aa-6eaacc747d01"
-					(reference "D23")
+					(reference "D27")
 					(unit 1)
 				)
@@
 			)
 		)
-		(property "Footprint" "FP-PTN0603-IPC_B"
+		(property "Footprint" "Vault:FP-PTN0603-IPC_B"
 			(at 76.2 175.26 0)
 			(hide yes)
@@
 			)
 		)
-		(property "Footprint" "SI5418DU-T1-GE3-Footprint-1"
+		(property "Footprint" "Vault:SI5418DU-T1-GE3-Footprint-1"
 			(at 162.56 114.3 0)
 			(hide yes)
@@
 			)
 		)
-		(property "Footprint" "FP-CSR1206-IPC_C"
+		(property "Footprint" "Vault:FP-CSR1206-IPC_C"
 			(at 60.96 109.22 0)
 			(hide yes)
@@
 			)
 		)
-		(property "Footprint" "RESC0402(1005)_L"
+		(property "Footprint" "Vault:RESC0402(1005)_L"
 			(at 76.2 139.7 0)
 			(hide yes)
@@
 		(in_pos_files yes)
 		(dnp no)
-		(property "Reference" "#PWR?"
+		(property "Reference" "#PWR092"
 			(at 129.54 78.74 0)
 			(hide yes)
@@
 			(project "LEARNSAT_POBOY_v3.2.0"
 				(path "/31302da5-a970-4b2b-aa05-afcd06cb9d09/7afe09a5-989f-4cf0-b7aa-6eaacc747d01"
-					(reference "#PWR?")
+					(reference "#PWR092")
 					(unit 1)
 				)
@@
 			)
 		)
-		(property "Footprint" "FP-C0805C-DN-IPC_A"
+		(property "Footprint" "Vault:FP-C0805C-DN-IPC_A"
 			(at 137.16 154.94 0)
 			(hide yes)
@@
 			)
 		)
-		(property "Footprint" "CAPC1608X90X40LL10T20"
+		(property "Footprint" "Vault:CAPC1608X90X40LL10T20"
 			(at 81.28 76.2 0)
 			(hide yes)
