File: LEARNSAT_PoBoI/12VPrimary.kicad_sch (KiCad schematic)
At the start: 17 parts, among them Q12 SI5418DU-T1-GE3, Q3 SI7164DP-T1-GE3, U13 INA219AIDCNR, U18 LTC4231IUD-2#TRPBF

Commit message: added footprints
Parts:
- C28: footprint CAPC1608X90X40LL10T20 -> Vault:CAPC1608X90X40LL10T20
- C33: footprint FP-C0805C-DN-IPC_A -> Vault:FP-C0805C-DN-IPC_A
- C34: footprint CAPC1608X90X35ML15T15 -> Vault:CAPC1608X90X35ML15T15
- D23: footprint ONSC-SOD-323-2-477-02_V -> Vault:ONSC-SOD-323-2-477-02_V
- Q12: footprint SI5418DU-T1-GE3-Footprint-1 -> Vault:SI5418DU-T1-GE3-Footprint-1
- Q3: footprint Vishay_S17-0173-SINGLE_MFG -> Vault:Vishay_S17-0173-SINGLE_MFG
- R15, R16: footprint FP-CRCW1210-e3-IPC_C -> Vault:FP-CRCW1210-e3-IPC_C
- R23, R25, R37: footprint RESC0402(1005)_L -> Vault:RESC0402(1005)_L
- R28: footprint FP-CSR1206-IPC_C -> Vault:FP-CSR1206-IPC_C
- R35: footprint FP-CRCW1206-e3-IPC_A -> Vault:FP-CRCW1206-e3-IPC_A
- R39: footprint FP-PTN0603-IPC_B -> Vault:FP-PTN0603-IPC_B
- R40: footprint FP-RT1206-IPC_C -> Vault:FP-RT1206-IPC_C
- U13: footprint FP-DCN0008A-IPC_A -> Vault:FP-DCN0008A-IPC_A
- U18: footprint FP-UD-12-05-08-1855-IPC_A -> Vault:FP-UD-12-05-08-1855-IPC_A
Changed lines of the file:
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@@
 			)
 		)
-		(property "Footprint" "FP-UD-12-05-08-1855-IPC_A"
+		(property "Footprint" "Vault:FP-UD-12-05-08-1855-IPC_A"
 			(at 101.6 134.62 0)
 			(hide yes)
@@
 			)
 		)
-		(property "Footprint" "FP-PTN0603-IPC_B"
+		(property "Footprint" "Vault:FP-PTN0603-IPC_B"
 			(at 81.28 175.26 0)
 			(hide yes)
@@
 			)
 		)
-		(property "Footprint" "FP-CRCW1206-e3-IPC_A"
+		(property "Footprint" "Vault:FP-CRCW1206-e3-IPC_A"
 			(at 81.28 157.48 0)
 			(hide yes)
@@
 			)
 		)
-		(property "Footprint" "CAPC1608X90X40LL10T20"
+		(property "Footprint" "Vault:CAPC1608X90X40LL10T20"
 			(at 86.36 76.2 0)
 			(hide yes)
@@
 			)
 		)
-		(property "Footprint" "CAPC1608X90X35ML15T15"
+		(property "Footprint" "Vault:CAPC1608X90X35ML15T15"
 			(at 114.3 43.18 0)
 			(hide yes)
@@
 			)
 		)
-		(property "Footprint" "SI5418DU-T1-GE3-Footprint-1"
+		(property "Footprint" "Vault:SI5418DU-T1-GE3-Footprint-1"
 			(at 167.64 114.3 0)
 			(hide yes)
@@
 			)
 		)
-		(property "Footprint" "FP-DCN0008A-IPC_A"
+		(property "Footprint" "Vault:FP-DCN0008A-IPC_A"
 			(at 99.06 63.5 0)
 			(hide yes)
@@
 			)
 		)
-		(property "Footprint" "FP-C0805C-DN-IPC_A"
+		(property "Footprint" "Vault:FP-C0805C-DN-IPC_A"
 			(at 142.24 154.94 0)
 			(hide yes)
@@
 			)
 		)
-		(property "Footprint" "RESC0402(1005)_L"
+		(property "Footprint" "Vault:RESC0402(1005)_L"
 			(at 66.04 93.98 0)
 			(hide yes)
@@
 			)
 		)
-		(property "Footprint" "FP-RT1206-IPC_C"
+		(property "Footprint" "Vault:FP-RT1206-IPC_C"
 			(at 81.28 193.04 0)
 			(hide yes)
@@
 			)
 		)
-		(property "Footprint" "RESC0402(1005)_L"
+		(property "Footprint" "Vault:RESC0402(1005)_L"
 			(at 81.28 139.7 0)
 			(hide yes)
@@
 			)
 		)
-		(property "Footprint" "FP-CRCW1210-e3-IPC_C"
+		(property "Footprint" "Vault:FP-CRCW1210-e3-IPC_C"
 			(at 134.62 48.26 0)
 			(hide yes)
@@
 			)
 		)
-		(property "Footprint" "FP-CRCW1210-e3-IPC_C"
+		(property "Footprint" "Vault:FP-CRCW1210-e3-IPC_C"
 			(at 144.78 48.26 0)
 			(hide yes)
@@
 			)
 		)
-		(property "Footprint" "RESC0402(1005)_L"
+		(property "Footprint" "Vault:RESC0402(1005)_L"
 			(at 83.82 93.98 0)
 			(hide yes)
@@
 			)
 		)
-		(property "Footprint" "ONSC-SOD-323-2-477-02_V"
+		(property "Footprint" "Vault:ONSC-SOD-323-2-477-02_V"
 			(at 170.18 160.02 0)
 			(hide yes)
@@
 			)
 		)
-		(property "Footprint" "FP-CSR1206-IPC_C"
+		(property "Footprint" "Vault:FP-CSR1206-IPC_C"
 			(at 66.04 109.22 0)
 			(hide yes)
@@
 			)
 		)
-		(property "Footprint" "Vishay_S17-0173-SINGLE_MFG"
+		(property "Footprint" "Vault:Vishay_S17-0173-SINGLE_MFG"
 			(at 127 129.54 0)
 			(hide yes)
