File: LEARNSAT_PoBoI/5VPrimary.kicad_sch (KiCad schematic)
At the start: 17 parts, among them Q1201 SI7164DP-T1-GE3, Q1202 SI5418DU-T1-GE3, U1201 INA219AIDCNR, U1202 LTC4231IUD-2#TRPBF

Commit message: Add files via upload
Parts:
- C38: renamed from C1202; footprint Capacitor_SMD:C_0603_1608Metric -> CAPC1608X90X35ML15T15
- C39: renamed from C1201; footprint Capacitor_SMD:C_0603_1608Metric -> CAPC1608X90X40LL10T20
- C43: renamed from C1203; footprint Capacitor_SMD:C_0805_2012Metric -> FP-C0805C-DN-IPC_A
- D24: renamed from D1201; footprint Diode_SMD:D_SOD-323 -> ONSC-SOD-323-2-477-02_V
- Q7: renamed from Q1201; footprint Package_SO:Vishay_PowerPAK_1212-8_Single -> Vishay_S17-0173-SINGLE_MFG
- Q9: renamed from Q1202; footprint Package_SO:Vishay_PowerPAK_1212-8_Single -> SI5418DU-T1-GE3-Footprint-1
- R43: renamed from R1208; footprint Resistor_SMD:R_1210_3225Metric -> FP-CRCW1210-e3-IPC_C
- R44: renamed from R1209; footprint Resistor_SMD:R_1210_3225Metric -> FP-CRCW1210-e3-IPC_C
- R49: renamed from R1207; footprint Resistor_SMD:R_0402_1005Metric -> RESC0402(1005)_L
- R50: renamed from R1201; footprint Resistor_SMD:R_0402_1005Metric -> RESC0402(1005)_L
- R51: renamed from R1202; footprint Resistor_SMD:R_1206_3216Metric -> FP-CSR1206-IPC_C
- R56: renamed from R1204; footprint Resistor_SMD:R_1206_3216Metric -> FP-CRCW1206-e3-IPC_A
- R57: renamed from R1203; footprint Resistor_SMD:R_0402_1005Metric -> RESC0402(1005)_L
- R58: renamed from R1206; footprint Resistor_SMD:R_1206_3216Metric -> FP-RT1206-IPC_C
- R59: renamed from R1205; footprint Resistor_SMD:R_0603_1608Metric -> FP-PTN0603-IPC_B
- U20: renamed from U1201; footprint INA219AIDCNR:SOT65P280X145-8N -> FP-DCN0008A-IPC_A
- U25: renamed from U1202; footprint LTC4231IUD-2_TRPBF:QFN50P300X300X80-13N -> FP-UD-12-05-08-1855-IPC_A

Commit message: added footprints
Parts:
- C38: footprint CAPC1608X90X35ML15T15 -> Vault:CAPC1608X90X35ML15T15
- C39: footprint CAPC1608X90X40LL10T20 -> Vault:CAPC1608X90X40LL10T20
- C43: footprint FP-C0805C-DN-IPC_A -> Vault:FP-C0805C-DN-IPC_A
- D24: footprint ONSC-SOD-323-2-477-02_V -> Vault:ONSC-SOD-323-2-477-02_V
- Q7: footprint Vishay_S17-0173-SINGLE_MFG -> Vault:Vishay_S17-0173-SINGLE_MFG
- Q9: footprint SI5418DU-T1-GE3-Footprint-1 -> Vault:SI5418DU-T1-GE3-Footprint-1
- R43, R44: footprint FP-CRCW1210-e3-IPC_C -> Vault:FP-CRCW1210-e3-IPC_C
- R49, R50, R57: footprint RESC0402(1005)_L -> Vault:RESC0402(1005)_L
- R51: footprint FP-CSR1206-IPC_C -> Vault:FP-CSR1206-IPC_C
- R56: footprint FP-CRCW1206-e3-IPC_A -> Vault:FP-CRCW1206-e3-IPC_A
- R58: footprint FP-RT1206-IPC_C -> Vault:FP-RT1206-IPC_C
- R59: footprint FP-PTN0603-IPC_B -> Vault:FP-PTN0603-IPC_B
- U20: footprint FP-DCN0008A-IPC_A -> Vault:FP-DCN0008A-IPC_A
- U25: footprint FP-UD-12-05-08-1855-IPC_A -> Vault:FP-UD-12-05-08-1855-IPC_A
Changed lines of the file:
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@@
 		(in_pos_files yes)
 		(dnp no)
-		(property "Reference" "#PWR?"
+		(property "Reference" "#PWR086"
 			(at 129.54 78.74 0)
 			(hide yes)
@@
 			(project "LEARNSAT_POBOY_v3.2.0"
 				(path "/31302da5-a970-4b2b-aa05-afcd06cb9d09/f2874a5c-bf0c-4149-b3d2-1179c2685763"
-					(reference "#PWR?")
+					(reference "#PWR086")
 					(unit 1)
 				)
@@
 			)
 		)
-		(property "Footprint" "FP-C0805C-DN-IPC_A"
+		(property "Footprint" "Vault:FP-C0805C-DN-IPC_A"
 			(at 137.16 154.94 0)
 			(hide yes)
@@
 			)
 		)
-		(property "Footprint" "SI5418DU-T1-GE3-Footprint-1"
+		(property "Footprint" "Vault:SI5418DU-T1-GE3-Footprint-1"
 			(at 162.56 114.3 0)
 			(hide yes)
@@
 			)
 		)
-		(property "Footprint" "FP-CSR1206-IPC_C"
+		(property "Footprint" "Vault:FP-CSR1206-IPC_C"
 			(at 60.96 109.22 0)
 			(hide yes)
@@
 			)
 		)
-		(property "Footprint" "ONSC-SOD-323-2-477-02_V"
+		(property "Footprint" "Vault:ONSC-SOD-323-2-477-02_V"
 			(at 165.1 157.48 0)
 			(hide yes)
@@
 			)
 		)
-		(property "Footprint" "CAPC1608X90X40LL10T20"
+		(property "Footprint" "Vault:CAPC1608X90X40LL10T20"
 			(at 81.28 76.2 0)
 			(hide yes)
@@
 		(in_pos_files yes)
 		(dnp no)
-		(property "Reference" "#PWR?"
+		(property "Reference" "#PWR087"
 			(at 139.7 78.74 0)
 			(hide yes)
@@
 			(project "LEARNSAT_POBOY_v3.2.0"
 				(path "/31302da5-a970-4b2b-aa05-afcd06cb9d09/f2874a5c-bf0c-4149-b3d2-1179c2685763"
-					(reference "#PWR?")
+					(reference "#PWR087")
 					(unit 1)
 				)
@@
 		(in_pos_files yes)
 		(dnp no)
-		(property "Reference" "#PWR?"
+		(property "Reference" "#PWR089"
 			(at 154.94 154.94 0)
 			(hide yes)
@@
 			(project "LEARNSAT_POBOY_v3.2.0"
 				(path "/31302da5-a970-4b2b-aa05-afcd06cb9d09/f2874a5c-bf0c-4149-b3d2-1179c2685763"
-					(reference "#PWR?")
+					(reference "#PWR089")
 					(unit 1)
 				)
@@
 		(in_pos_files yes)
 		(dnp no)
-		(property "Reference" "#PWR?"
+		(property "Reference" "#PWR085"
 			(at 121.92 35.56 0)
 			(hide yes)
@@
 			(project "LEARNSAT_POBOY_v3.2.0"
 				(path "/31302da5-a970-4b2b-aa05-afcd06cb9d09/f2874a5c-bf0c-4149-b3d2-1179c2685763"
-					(reference "#PWR?")
+					(reference "#PWR085")
 					(unit 1)
 				)
@@
 			)
 		)
-		(property "Footprint" "FP-RT1206-IPC_C"
+		(property "Footprint" "Vault:FP-RT1206-IPC_C"
 			(at 76.2 193.04 0)
 			(hide yes)
@@
 			)
 		)
-		(property "Footprint" "FP-CRCW1210-e3-IPC_C"
+		(property "Footprint" "Vault:FP-CRCW1210-e3-IPC_C"
 			(at 129.54 48.26 0)
 			(hide yes)
@@
 			)
 		)
-		(property "Footprint" "FP-CRCW1206-e3-IPC_A"
+		(property "Footprint" "Vault:FP-CRCW1206-e3-IPC_A"
 			(at 76.2 157.48 0)
 			(hide yes)
@@
 			)
 		)
-		(property "Footprint" "RESC0402(1005)_L"
+		(property "Footprint" "Vault:RESC0402(1005)_L"
 			(at 76.2 139.7 0)
 			(hide yes)
@@
 			)
 		)
-		(property "Footprint" "RESC0402(1005)_L"
+		(property "Footprint" "Vault:RESC0402(1005)_L"
 			(at 78.74 93.98 0)
 			(hide yes)
@@
 			)
 		)
-		(property "Footprint" "CAPC1608X90X35ML15T15"
+		(property "Footprint" "Vault:CAPC1608X90X35ML15T15"
 			(at 109.22 43.18 0)
 			(hide yes)
@@
 			)
 		)
-		(property "Footprint" "FP-UD-12-05-08-1855-IPC_A"
+		(property "Footprint" "Vault:FP-UD-12-05-08-1855-IPC_A"
 			(at 96.52 134.62 0)
 			(hide yes)
@@
 			)
 		)
-		(property "Footprint" "FP-DCN0008A-IPC_A"
+		(property "Footprint" "Vault:FP-DCN0008A-IPC_A"
 			(at 93.98 63.5 0)
 			(hide yes)
@@
 			)
 		)
-		(property "Footprint" "RESC0402(1005)_L"
+		(property "Footprint" "Vault:RESC0402(1005)_L"
 			(at 60.96 93.98 0)
 			(hide yes)
@@
 			)
 		)
-		(property "Footprint" "Vishay_S17-0173-SINGLE_MFG"
+		(property "Footprint" "Vault:Vishay_S17-0173-SINGLE_MFG"
 			(at 121.92 129.54 0)
 			(hide yes)
@@
 		(in_pos_files yes)
 		(dnp no)
-		(property "Reference" "#PWR?"
+		(property "Reference" "#PWR088"
 			(at 144.78 167.64 0)
 			(hide yes)
@@
 			(project "LEARNSAT_POBOY_v3.2.0"
 				(path "/31302da5-a970-4b2b-aa05-afcd06cb9d09/f2874a5c-bf0c-4149-b3d2-1179c2685763"
-					(reference "#PWR?")
+					(reference "#PWR088")
 					(unit 1)
 				)
@@
 			)
 		)
-		(property "Footprint" "FP-PTN0603-IPC_B"
+		(property "Footprint" "Vault:FP-PTN0603-IPC_B"
 			(at 76.2 175.26 0)
 			(hide yes)
@@
 			)
 		)
-		(property "Footprint" "FP-CRCW1210-e3-IPC_C"
+		(property "Footprint" "Vault:FP-CRCW1210-e3-IPC_C"
 			(at 139.7 48.26 0)
 			(hide yes)
@@
 		(in_pos_files yes)
 		(dnp no)
-		(property "Reference" "#PWR?"
+		(property "Reference" "#PWR090"
 			(at 162.56 167.64 0)
 			(hide yes)
@@
 			(project "LEARNSAT_POBOY_v3.2.0"
 				(path "/31302da5-a970-4b2b-aa05-afcd06cb9d09/f2874a5c-bf0c-4149-b3d2-1179c2685763"
-					(reference "#PWR?")
+					(reference "#PWR090")
 					(unit 1)
 				)
