File: LEARNSAT_PoBoI/MemoryLatch.kicad_sch (KiCad schematic)
At the start: 1 part, among them U1501 SN74LVC1G373DCKR

Commit message: Add files via upload
Parts:
- U23: renamed from U1501; footprint SN74LVC1G373DCKR:SOT65P210X110-6N -> DCK0006A_M

Commit message: added footprints
Parts:
- U23: footprint DCK0006A_M -> Vault:DCK0006A_M
Changed lines of the file:
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@@
 		(in_pos_files yes)
 		(dnp no)
-		(property "Reference" "#PWR?"
+		(property "Reference" "#PWR0109"
 			(at 81.28 109.22 0)
 			(hide yes)
@@
 			(project "LEARNSAT_POBOY_v3.2.0"
 				(path "/31302da5-a970-4b2b-aa05-afcd06cb9d09/af482a7d-1f10-48c9-bdaf-5889a5ffb8a7"
-					(reference "#PWR?")
+					(reference "#PWR0109")
 					(unit 1)
 				)
@@
 		(in_pos_files yes)
 		(dnp no)
-		(property "Reference" "#PWR?"
+		(property "Reference" "#PWR0110"
 			(at 137.16 119.38 0)
 			(hide yes)
@@
 			(project "LEARNSAT_POBOY_v3.2.0"
 				(path "/31302da5-a970-4b2b-aa05-afcd06cb9d09/af482a7d-1f10-48c9-bdaf-5889a5ffb8a7"
-					(reference "#PWR?")
+					(reference "#PWR0110")
 					(unit 1)
 				)
@@
 			)
 		)
-		(property "Footprint" "DCK0006A_M"
+		(property "Footprint" "Vault:DCK0006A_M"
 			(at 109.22 104.14 0)
 			(hide yes)
