File: LEARNSAT_PoBoI/STM32.kicad_sch (KiCad schematic)
At the start: 24 parts, among them U17 LP5907SNX-3.3, U21 74AC14MTCX, U22 LTC4304CMS#PBF, U26 ISL3259EIRZ, U6 STM32F103RET6, Y1 ABS07-166-32.768KHZ-T

Commit message: added footprints
Parts:
- C21, C23: footprint FP-CC0201-BA-IPC_A -> Vault:FP-CC0201-BA-IPC_A
- C30, C31, C42, C44, C46, C47: footprint FP-C0603-CJ-MFG -> Vault:FP-C0603-CJ-MFG
- C35: footprint CAPC1608X94X35NL15T15 -> Vault:CAPC1608X94X35NL15T15
- C40, C45: footprint FP-GRM033-0_03-IPC_A -> Vault:FP-GRM033-0_03-IPC_A
- D10, D9: footprint 1N4148WX-TP-Footprint-1 -> Vault:1N4148WX-TP-Footprint-1
- R22: footprint RESC0402(1005)_L -> Vault:RESC0402(1005)_L
- R36: footprint RESC1005X40X25NL05T10 -> Vault:RESC1005X40X25NL05T10
- R38: footprint RESC3216X60X45ML15T20 -> Vault:RESC3216X60X45ML15T20
- R48: footprint RESC1608X55X25ML10T15 -> Vault:RESC1608X55X25ML10T15
- R60: footprint RESC0603(1608)_L -> Vault:RESC0603(1608)_L
- U17: footprint TI-DQN4-480X480TP_V -> Vault:TI-DQN4-480X480TP_V
- U21: footprint FP-948G-MFG -> Vault:FP-948G-MFG
- U22: footprint LTC4304CMS#PBF-Footprint-1 -> Vault:LTC4304CMS#PBF-Footprint-1
- U26: footprint ISL3259EIRZ-Footprint-1 -> Vault:ISL3259EIRZ-Footprint-1
- U6: footprint STM-LQFP64_N -> Vault:STM-LQFP64_N
- Y1: footprint EPSON-FC-135_V -> Vault:EPSON-FC-135_V
Changed lines of the file:
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@@
 		(in_pos_files yes)
 		(dnp no)
-		(property "Reference" "#PWR?"
+		(property "Reference" "#PWR021"
 			(at 58.42 162.56 0)
 			(hide yes)
@@
 			(project "LEARNSAT_POBOY_v3.2.0"
 				(path "/31302da5-a970-4b2b-aa05-afcd06cb9d09/9cfff8c1-41d5-443e-a4f1-1edb2a27fa2d"
-					(reference "#PWR?")
+					(reference "#PWR021")
 					(unit 1)
 				)
@@
 			)
 		)
-		(property "Footprint" "FP-CC0201-BA-IPC_A"
+		(property "Footprint" "Vault:FP-CC0201-BA-IPC_A"
 			(at 15.24 190.5 0)
 			(hide yes)
@@
 			)
 		)
-		(property "Footprint" "STM-LQFP64_N"
+		(property "Footprint" "Vault:STM-LQFP64_N"
 			(at 111.76 38.1 0)
 			(hide yes)
@@
 			)
 		)
-		(property "Footprint" "CAPC1608X94X35NL15T15"
+		(property "Footprint" "Vault:CAPC1608X94X35NL15T15"
 			(at 180.34 172.72 0)
 			(hide yes)
@@
 			)
 		)
-		(property "Footprint" "STM-LQFP64_N"
+		(property "Footprint" "Vault:STM-LQFP64_N"
 			(at 109.22 139.7 0)
 			(hide yes)
@@
 			)
 		)
-		(property "Footprint" "1N4148WX-TP-Footprint-1"
+		(property "Footprint" "Vault:1N4148WX-TP-Footprint-1"
 			(at 35.56 43.18 0)
 			(hide yes)
@@
 			)
 		)
-		(property "Footprint" "FP-GRM033-0_03-IPC_A"
+		(property "Footprint" "Vault:FP-GRM033-0_03-IPC_A"
 			(at 215.9 114.3 0)
 			(hide yes)
@@
 		(in_pos_files yes)
 		(dnp no)
-		(property "Reference" "#PWR?"
+		(property "Reference" "#PWR034"
 			(at 215.9 121.92 0)
 			(hide yes)
@@
 			(project "LEARNSAT_POBOY_v3.2.0"
 				(path "/31302da5-a970-4b2b-aa05-afcd06cb9d09/9cfff8c1-41d5-443e-a4f1-1edb2a27fa2d"
-					(reference "#PWR?")
+					(reference "#PWR034")
 					(unit 1)
 				)
@@
 			)
 		)
-		(property "Footprint" "FP-948G-MFG"
+		(property "Footprint" "Vault:FP-948G-MFG"
 			(at 30.48 63.5 0)
 			(hide yes)
@@
 			)
 		)
-		(property "Footprint" "FP-C0603-CJ-MFG"
+		(property "Footprint" "Vault:FP-C0603-CJ-MFG"
 			(at 208.28 73.66 0)
 			(hide yes)
@@
 		(in_pos_files yes)
 		(dnp no)
-		(property "Reference" "#PWR?"
+		(property "Reference" "#PWR029"
 			(at 180.34 180.34 0)
 			(hide yes)
@@
 			(project "LEARNSAT_POBOY_v3.2.0"
 				(path "/31302da5-a970-4b2b-aa05-afcd06cb9d09/9cfff8c1-41d5-443e-a4f1-1edb2a27fa2d"
-					(reference "#PWR?")
+					(reference "#PWR029")
 					(unit 1)
 				)
@@
 		(in_pos_files yes)
 		(dnp no)
-		(property "Reference" "#PWR?"
+		(property "Reference" "#PWR020"
 			(at 55.88 198.12 0)
 			(hide yes)
@@
 			(project "LEARNSAT_POBOY_v3.2.0"
 				(path "/31302da5-a970-4b2b-aa05-afcd06cb9d09/9cfff8c1-41d5-443e-a4f1-1edb2a27fa2d"
-					(reference "#PWR?")
+					(reference "#PWR020")
 					(unit 1)
 				)
@@
 			)
 		)
-		(property "Footprint" "EPSON-FC-135_V"
+		(property "Footprint" "Vault:EPSON-FC-135_V"
 			(at 190.5 109.22 0)
 			(hide yes)
@@
 		(in_pos_files yes)
 		(dnp no)
-		(property "Reference" "#PWR?"
+		(property "Reference" "#PWR019"
 			(at 15.24 200.66 0)
 			(hide yes)
@@
 			(project "LEARNSAT_POBOY_v3.2.0"
 				(path "/31302da5-a970-4b2b-aa05-afcd06cb9d09/9cfff8c1-41d5-443e-a4f1-1edb2a27fa2d"
-					(reference "#PWR?")
+					(reference "#PWR019")
 					(unit 1)
 				)
@@
 			)
 		)
-		(property "Footprint" "RESC0603(1608)_L"
+		(property "Footprint" "Vault:RESC0603(1608)_L"
 			(at 76.2 149.86 0)
 			(hide yes)
@@
 			)
 		)
-		(property "Footprint" "RESC1608X55X25ML10T15"
+		(property "Footprint" "Vault:RESC1608X55X25ML10T15"
 			(at 185.42 139.7 0)
 			(hide yes)
@@
 			)
 		)
-		(property "Footprint" "1N4148WX-TP-Footprint-1"
+		(property "Footprint" "Vault:1N4148WX-TP-Footprint-1"
 			(at 35.56 50.8 0)
 			(hide yes)
@@
 		(in_pos_files yes)
 		(dnp no)
-		(property "Reference" "#PWR?"
+		(property "Reference" "#PWR033"
 			(at 208.28 81.28 0)
 			(hide yes)
@@
 			(project "LEARNSAT_POBOY_v3.2.0"
 				(path "/31302da5-a970-4b2b-aa05-afcd06cb9d09/9cfff8c1-41d5-443e-a4f1-1edb2a27fa2d"
-					(reference "#PWR?")
+					(reference "#PWR033")
 					(unit 1)
 				)
@@
 			)
 		)
-		(property "Footprint" "FP-GRM033-0_03-IPC_A"
+		(property "Footprint" "Vault:FP-GRM033-0_03-IPC_A"
 			(at 170.18 114.3 0)
 			(hide yes)
@@
 		(in_pos_files yes)
 		(dnp no)
-		(property "Reference" "#PWR?"
+		(property "Reference" "#PWR024"
 			(at 124.46 200.66 0)
 			(hide yes)
@@
 			(project "LEARNSAT_POBOY_v3.2.0"
 				(path "/31302da5-a970-4b2b-aa05-afcd06cb9d09/9cfff8c1-41d5-443e-a4f1-1edb2a27fa2d"
-					(reference "#PWR?")
+					(reference "#PWR024")
 					(unit 1)
 				)
@@
 			)
 		)
-		(property "Footprint" "FP-C0603-CJ-MFG"
+		(property "Footprint" "Vault:FP-C0603-CJ-MFG"
 			(at 193.04 48.26 0)
 			(hide yes)
@@
 		(in_pos_files yes)
 		(dnp no)
-		(property "Reference" "#PWR?"
+		(property "Reference" "#PWR027"
 			(at 177.8 55.88 0)
 			(hide yes)
@@
 			(project "LEARNSAT_POBOY_v3.2.0"
 				(path "/31302da5-a970-4b2b-aa05-afcd06cb9d09/9cfff8c1-41d5-443e-a4f1-1edb2a27fa2d"
-					(reference "#PWR?")
+					(reference "#PWR027")
 					(unit 1)
 				)
@@
 		(in_pos_files yes)
 		(dnp no)
-		(property "Reference" "#PWR?"
+		(property "Reference" "#PWR025"
 			(at 139.7 165.1 0)
 			(hide yes)
@@
 			(project "LEARNSAT_POBOY_v3.2.0"
 				(path "/31302da5-a970-4b2b-aa05-afcd06cb9d09/9cfff8c1-41d5-443e-a4f1-1edb2a27fa2d"
-					(reference "#PWR?")
+					(reference "#PWR025")
 					(unit 1)
 				)
@@
 		(in_pos_files yes)
 		(dnp no)
-		(property "Reference" "#PWR?"
+		(property "Reference" "#PWR028"
 			(at 177.8 81.28 0)
 			(hide yes)
@@
 			(project "LEARNSAT_POBOY_v3.2.0"
 				(path "/31302da5-a970-4b2b-aa05-afcd06cb9d09/9cfff8c1-41d5-443e-a4f1-1edb2a27fa2d"
-					(reference "#PWR?")
+					(reference "#PWR028")
 					(unit 1)
 				)
@@
 			)
 		)
-		(property "Footprint" "FP-C0603-CJ-MFG"
+		(property "Footprint" "Vault:FP-C0603-CJ-MFG"
 			(at 177.8 73.66 0)
 			(hide yes)
@@
 			)
 		)
-		(property "Footprint" "FP-CC0201-BA-IPC_A"
+		(property "Footprint" "Vault:FP-CC0201-BA-IPC_A"
 			(at 63.5 190.5 0)
 			(hide yes)
@@
 		(in_pos_files yes)
 		(dnp no)
-		(property "Reference" "#PWR?"
+		(property "Reference" "#PWR032"
 			(at 208.28 55.88 0)
 			(hide yes)
@@
 			(project "LEARNSAT_POBOY_v3.2.0"
 				(path "/31302da5-a970-4b2b-aa05-afcd06cb9d09/9cfff8c1-41d5-443e-a4f1-1edb2a27fa2d"
-					(reference "#PWR?")
+					(reference "#PWR032")
 					(unit 1)
 				)
@@
 			)
 		)
-		(property "Footprint" "TI-DQN4-480X480TP_V"
+		(property "Footprint" "Vault:TI-DQN4-480X480TP_V"
 			(at 25.4 187.96 0)
 			(hide yes)
@@
 			)
 		)
-		(property "Footprint" "FP-C0603-CJ-MFG"
+		(property "Footprint" "Vault:FP-C0603-CJ-MFG"
 			(at 208.28 48.26 0)
 			(hide yes)
@@
 			)
 		)
-		(property "Footprint" "LTC4304CMS#PBF-Footprint-1"
+		(property "Footprint" "Vault:LTC4304CMS#PBF-Footprint-1"
 			(at 180.34 149.86 0)
 			(hide yes)
@@
 			)
 		)
-		(property "Footprint" "RESC3216X60X45ML15T20"
+		(property "Footprint" "Vault:RESC3216X60X45ML15T20"
 			(at 165.1 162.56 0)
 			(hide yes)
@@
 			)
 		)
-		(property "Footprint" "RESC0402(1005)_L"
+		(property "Footprint" "Vault:RESC0402(1005)_L"
 			(at 124.46 185.42 0)
 			(hide yes)
@@
 			)
 		)
-		(property "Footprint" "FP-C0603-CJ-MFG"
+		(property "Footprint" "Vault:FP-C0603-CJ-MFG"
 			(at 193.04 73.66 0)
 			(hide yes)
@@
 			)
 		)
-		(property "Footprint" "FP-C0603-CJ-MFG"
+		(property "Footprint" "Vault:FP-C0603-CJ-MFG"
 			(at 177.8 48.26 0)
 			(hide yes)
@@
 		(in_pos_files yes)
 		(dnp no)
-		(property "Reference" "#PWR?"
+		(property "Reference" "#PWR022"
 			(at 60.96 114.3 0)
 			(hide yes)
@@
 			(project "LEARNSAT_POBOY_v3.2.0"
 				(path "/31302da5-a970-4b2b-aa05-afcd06cb9d09/9cfff8c1-41d5-443e-a4f1-1edb2a27fa2d"
-					(reference "#PWR?")
+					(reference "#PWR022")
 					(unit 1)
 				)
@@
 		(in_pos_files yes)
 		(dnp no)
-		(property "Reference" "#PWR?"
+		(property "Reference" "#PWR026"
 			(at 170.18 121.92 0)
 			(hide yes)
@@
 			(project "LEARNSAT_POBOY_v3.2.0"
 				(path "/31302da5-a970-4b2b-aa05-afcd06cb9d09/9cfff8c1-41d5-443e-a4f1-1edb2a27fa2d"
-					(reference "#PWR?")
+					(reference "#PWR026")
 					(unit 1)
 				)
@@
 		(in_pos_files yes)
 		(dnp no)
-		(property "Reference" "#PWR?"
+		(property "Reference" "#PWR030"
 			(at 193.04 55.88 0)
 			(hide yes)
@@
 			(project "LEARNSAT_POBOY_v3.2.0"
 				(path "/31302da5-a970-4b2b-aa05-afcd06cb9d09/9cfff8c1-41d5-443e-a4f1-1edb2a27fa2d"
-					(reference "#PWR?")
+					(reference "#PWR030")
 					(unit 1)
 				)
@@
 			)
 		)
-		(property "Footprint" "ISL3259EIRZ-Footprint-1"
+		(property "Footprint" "Vault:ISL3259EIRZ-Footprint-1"
 			(at 35.56 157.48 0)
 			(hide yes)
@@
 			)
 		)
-		(property "Footprint" "RESC1005X40X25NL05T10"
+		(property "Footprint" "Vault:RESC1005X40X25NL05T10"
 			(at 106.68 180.34 0)
 			(hide yes)
@@
 		(in_pos_files yes)
 		(dnp no)
-		(property "Reference" "#PWR?"
+		(property "Reference" "#PWR031"
 			(at 193.04 81.28 0)
 			(hide yes)
@@
 			(project "LEARNSAT_POBOY_v3.2.0"
 				(path "/31302da5-a970-4b2b-aa05-afcd06cb9d09/9cfff8c1-41d5-443e-a4f1-1edb2a27fa2d"
-					(reference "#PWR?")
+					(reference "#PWR031")
 					(unit 1)
 				)
@@
 		(in_pos_files yes)
 		(dnp no)
-		(property "Reference" "#PWR?"
+		(property "Reference" "#PWR023"
 			(at 63.5 198.12 0)
 			(hide yes)
@@
 			(project "LEARNSAT_POBOY_v3.2.0"
 				(path "/31302da5-a970-4b2b-aa05-afcd06cb9d09/9cfff8c1-41d5-443e-a4f1-1edb2a27fa2d"
-					(reference "#PWR?")
+					(reference "#PWR023")
 					(unit 1)
 				)
@@
 		(in_pos_files yes)
 		(dnp no)
-		(property "Reference" "#PWR?"
+		(property "Reference" "#PWR035"
 			(at 220.98 160.02 0)
 			(hide yes)
@@
 			(project "LEARNSAT_POBOY_v3.2.0"
 				(path "/31302da5-a970-4b2b-aa05-afcd06cb9d09/9cfff8c1-41d5-443e-a4f1-1edb2a27fa2d"
-					(reference "#PWR?")
+					(reference "#PWR035")
 					(unit 1)
 				)
