File: LEARNSAT_PoBoI/LEARNSAT_POBOY_v3.2.0.kicad_pcb (KiCad board)
At the start: 4 copper layers, 90.2 x 95.8 mm, 471 parts, among them J1 FTSH-105-01-L-DV-K-P-TR, J5 FTSH-105-01-L-DV-K-P-TR, P1 22-28-4036, Q1 SI7164DP-T1-GE3, Q10 SI5418DU-T1-GE3, Q11 SI7164DP-T1-GE3, Q12 SI5418DU-T1-GE3, Q13 SI5418DU-T1-GE3, Q13 SI7164DP-T1-GE3, Q14 SI5418DU-T1-GE3, Q14 SI7164DP-T1-GE3, Q15 SI7164DP-T1-GE3, Q16 SI5418DU-T1-GE3, Q17 SI7164DP-T1-GE3, Q18 SI5418DU-T1-GE3, Q19 SI7164DP-T1-GE3, Q2 SI7164DP-T1-GE3, Q20 SI5418DU-T1-GE3, Q20 SI7164DP-T1-GE3, Q21 SI7164DP-T1-GE3, Q22 SI5418DU-T1-GE3, Q23 SI7164DP-T1-GE3, Q24 SI5418DU-T1-GE3, Q3 SI7164DP-T1-GE3, Q4 SI5418DU-T1-GE3, Q5 SI5418DU-T1-GE3, Q6 SI7164DP-T1-GE3, Q7 SI7164DP-T1-GE3, Q8 SI5418DU-T1-GE3, Q9 SI5418DU-T1-GE3, SW1 B3U-1000P, SW2 B3U-1000P, SW3 TS04-66-43-BK-100-SMT, U1 MAX6746KA29+T, U1 STM32F103RET6, U10 LM2622MMX-ADJ/NOPB, U11 LM2622MMX-ADJ/NOPB, U12 INA219AIDCNR, U13 INA219AIDCNR, U14 INA219AIDCNR, U15 LTC4231IUD-2#TRPBF, U16 LTC4231IUD-2#TRPBF, U17 LP5907SNX-3.3, U18 LP5907SNX-3.3, U18 LTC4231IUD-2#TRPBF, U19 INA219AIDCNR, U2 SN74AUP1G08QDCKRQ1, U20 INA219AIDCNR, U21 74AC14MTCX, U22 LTC4231IUD-2#TRPBF, U22 LTC4304CMS#PBF, U23 INA219AIDCNR, U23 SN74LVC1G373DCKR, U24 LTC4231IUD-2#TRPBF, U25 INA219AIDCNR, U25 LTC4231IUD-2#TRPBF, U26 ISL3259EIRZ, U26 LTC4231IUD-2#TRPBF, U27 INA219AIDCNR, U28 LTC4231IUD-2#TRPBF, U29 INA219AIDCNR, U29 LTC4231IUD-2#TRPBF, U3 MAX6746KA29+T, U30 INA219AIDCNR, U30 LTC4231IUD-2#TRPBF, U31 INA219AIDCNR, U32 LTC4231IUD-2#TRPBF, U33 INA219AIDCNR, U34 MAX6746KA29+T, U35 MAX6746KA29+T, U36 SN74AUP1G08QDCKRQ1, U37 SN74AUP1G08QDCKRQ1, U38 LTC4304CMS#PBF, U39 74AC14MTCX, U4 SN74AUP1G08QDCKRQ1, U40 SN74LVC1G373DCKR, U41 ISL3259EIRZ, U5 LT1616ES6#TRMPBF, U50 LM2622MMX-ADJ/NOPB, U51 LM2622MMX-ADJ/NOPB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

Commit message: routed 12VPrimary
Parts:
- moved Q3 114.7 mm to (206.3, 89.9)
- moved R40 107.5 mm to (221.0, 92.4)
- moved U18 105.7 mm to (220.1, 87.9)
- moved R16 97.8 mm to (219.8, 77.7), turned to -90 degrees
- moved C28 96.4 mm to (207.3, 79.0), turned to 90 degrees
- moved C33 95.5 mm to (220.2, 82.9), turned to 180 degrees
- moved U13 94.9 mm to (211.7, 79.1)
- moved R35 94.5 mm to (213.6, 89.4)
- moved R37 93.2 mm to (215.1, 86.9), turned to -90 degrees
- moved R15 93.1 mm to (216.3, 77.7), turned to -90 degrees
- moved D23 91.9 mm to (216.5, 85.6), turned to -90 degrees
- moved R25 90.1 mm to (210.3, 82.3), turned to 90 degrees
- moved C34 88.7 mm to (212.5, 75.4)
- moved R39 88.2 mm to (216.9, 92.4)
- moved R23 87.9 mm to (208.8, 82.3), turned to 90 degrees
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Routing:
- net GND: track 173.8 -> 213.6 mm, vias 15 -> 17
- net Net-(Q12-S_1): track 0.00 -> 23.0 mm, vias 0 -> 2
- net 3V3: track 37.6 -> 58.6 mm, vias 2 -> 4
- net Net-(Q3-D): track 0.00 -> 20.4 mm
- net Net-(Q12-G): track 0.00 -> 16.7 mm, vias 0 -> 2
- net Net-(U13-IN+): track 0.00 -> 9.24 mm
- net Net-(U13-IN-): track 0.00 -> 8.48 mm
- net 12V: track 6.92 -> 14.7 mm
- net Net-(U18-UVL): track 0.00 -> 7.57 mm
- net SCL: track 14.2 -> 21.6 mm
- net Net-(U18-UVH): track 0.00 -> 7.30 mm
- net Net-(U18-TIMER): track 0.00 -> 6.13 mm
- net Net-(U18-OV): track 0.00 -> 5.04 mm
- net Net-(U18-GNDSW): track 0.00 -> 3.90 mm
- net SDA: track 15.5 -> 19.1 mm
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Other:
- board text added: "12VPrimary"
