File: LEARNSAT_PoBoI/12V_BOOST.kicad_sch (KiCad schematic)
At the start: 18 parts, among them U10 LM2622MMX-ADJ/NOPB, U11 LM2622MMX-ADJ/NOPB

Commit message: Small global net changes
Connections:
- net VBatt Primary: now reaches Cin1.1, L5.1, U10.6 (VIN)
- net VBatt Primary: now also Cin2.1, L6.1, U11.6 (VIN)
- net ???: now reaches Cout2.1, D19.1 (C), RFB4.2
- net ???: now also Cout1.1, D20.1 (C), RFB1.2

Commit message: Replaced local nets with global and left local nets intact
Other:
- note removed: "VBatt Primary"
Changed lines of the file:
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@@
 	(generator_version "10.0")
 	(paper "A")
-	(text "VBatt Primary"
-		(exclude_from_sim no)
-		(at 30.48 121.92 0)
-		(effects
-			(font
-				(size 1.27 1.27)
-			)
-			(justify left bottom)
-		)
-	)
-	(text "VBatt Primary"
-		(exclude_from_sim no)
-		(at 25.4 35.56 0)
-		(effects
-			(font
-				(size 1.27 1.27)
-			)
-			(justify left bottom)
-		)
-	)
 	(junction
 		(at 55.88 144.78)

Commit message: Added footprints
Parts:
- Cc301: renamed from Cc1; footprint FP-C0402-BB-MFG -> Capacitor_SMD:C_0402_1005Metric
- Cc302: renamed from Cc2; footprint FP-C0402-BB-MFG -> Capacitor_SMD:C_0402_1005Metric
- Cin301: renamed from Cin2; footprint FP-CL31-IPC_A -> Capacitor_SMD:C_1206_3216Metric
- Cin302: renamed from Cin1; footprint FP-CL31-IPC_A -> Capacitor_SMD:C_1206_3216Metric
- Cout301: renamed from Cout1; footprint FP-CL31-IPC_A -> Capacitor_SMD:C_1206_3216Metric
- Cout302: renamed from Cout2; footprint FP-CL31-IPC_A -> Capacitor_SMD:C_1206_3216Metric
- D301: renamed from D20; footprint FP-502-01-MFG -> Diode_SMD:D_SOD-123
- D302: renamed from D19; footprint FP-502-01-MFG -> Diode_SMD:D_SOD-123
- L301: renamed from L6; footprint FP-MLZ1608-IPC_C -> Inductor_SMD:L_0603_1608Metric
- L302: renamed from L5; footprint FP-MLZ1608-IPC_C -> Inductor_SMD:L_0603_1608Metric
- RFB301: renamed from RFB2; footprint FP-ERJ3EK-MFG -> Resistor_SMD:R_0603_1608Metric
- RFB302: renamed from RFB1; footprint RESC3216X70X50NL05T20 -> Resistor_SMD:R_1206_3216Metric
- RFB303: renamed from RFB3; footprint FP-ERJ3EK-MFG -> Resistor_SMD:R_0603_1608Metric
- RFB304: renamed from RFB4; footprint RESC3216X70X50NL05T20 -> Resistor_SMD:R_1206_3216Metric
- Rc301: renamed from Rc1; footprint RESC1005X40X25ML05T05 -> Resistor_SMD:R_0402_1005Metric
- Rc302: renamed from Rc2; footprint RESC1005X40X25ML05T05 -> Resistor_SMD:R_0402_1005Metric
- U301: renamed from U11; footprint DGK0008A_M -> LM2622MMX-ADJ_NOPB:SOP65P490X110-8N
- U302: renamed from U10; footprint DGK0008A_M -> LM2622MMX-ADJ_NOPB:SOP65P490X110-8N
Connections:
- net ???: no longer names the net of Cout302.1, D302.1 (C), RFB304.2
- net ???: no longer Cout301.1, D301.1 (C), RFB302.2
- net VBatt Primary: no longer names the net of Cin302.1, L302.1, U302.6 (VIN)
- net VBatt Primary: no longer Cin301.1, L301.1, U301.6 (VIN)
- new net: Cin301.1, L301.1, U301.6 (VIN)
- new net: Cout301.1, D301.1 (C), RFB302.2
Other:
- note added: "VBatt Primary"

Commit message: Add files via upload
Parts:
- Cc1: renamed from Cc301; footprint Capacitor_SMD:C_0402_1005Metric -> FP-C0402-BB-MFG
- Cc2: renamed from Cc302; footprint Capacitor_SMD:C_0402_1005Metric -> FP-C0402-BB-MFG
- Cin1: renamed from Cin302; footprint Capacitor_SMD:C_1206_3216Metric -> FP-CL31-IPC_A
- Cin2: renamed from Cin301; footprint Capacitor_SMD:C_1206_3216Metric -> FP-CL31-IPC_A
- Cout1: renamed from Cout301; footprint Capacitor_SMD:C_1206_3216Metric -> FP-CL31-IPC_A
- Cout2: renamed from Cout302; footprint Capacitor_SMD:C_1206_3216Metric -> FP-CL31-IPC_A
- D19: renamed from D302; footprint Diode_SMD:D_SOD-123 -> FP-502-01-MFG
- D20: renamed from D301; footprint Diode_SMD:D_SOD-123 -> FP-502-01-MFG
- L5: renamed from L302; footprint Inductor_SMD:L_0603_1608Metric -> FP-MLZ1608-IPC_C
- L6: renamed from L301; footprint Inductor_SMD:L_0603_1608Metric -> FP-MLZ1608-IPC_C
- RFB1: renamed from RFB302; footprint Resistor_SMD:R_1206_3216Metric -> RESC3216X70X50NL05T20
- RFB2: renamed from RFB301; footprint Resistor_SMD:R_0603_1608Metric -> FP-ERJ3EK-MFG
- RFB3: renamed from RFB303; footprint Resistor_SMD:R_0603_1608Metric -> FP-ERJ3EK-MFG
- RFB4: renamed from RFB304; footprint Resistor_SMD:R_1206_3216Metric -> RESC3216X70X50NL05T20
- Rc1: renamed from Rc301; footprint Resistor_SMD:R_0402_1005Metric -> RESC1005X40X25ML05T05
- Rc2: renamed from Rc302; footprint Resistor_SMD:R_0402_1005Metric -> RESC1005X40X25ML05T05
- U10: renamed from U302; footprint LM2622MMX-ADJ_NOPB:SOP65P490X110-8N -> DGK0008A_M
- U11: renamed from U301; footprint LM2622MMX-ADJ_NOPB:SOP65P490X110-8N -> DGK0008A_M
Connections:
- net VBatt Primary: now reaches Cin1.1, L5.1, U10.6 (VIN)
- net VBatt Primary: now also Cin2.1, L6.1, U11.6 (VIN)
- net ???: now reaches Cout2.1, D19.1 (C), RFB4.2
- net ???: now also Cout1.1, D20.1 (C), RFB1.2
Other:
- note removed: "VBatt Primary"

Commit message: added footprints
Parts:
- Cc1, Cc2: footprint FP-C0402-BB-MFG -> Vault:FP-C0402-BB-MFG
- Cin1, Cin2, Cout1, Cout2: footprint FP-CL31-IPC_A -> Vault:FP-CL31-IPC_A
- D19, D20: footprint FP-502-01-MFG -> Vault:FP-502-01-MFG
- L5, L6: footprint FP-MLZ1608-IPC_C -> Vault:FP-MLZ1608-IPC_C
- RFB1, RFB4: footprint RESC3216X70X50NL05T20 -> Vault:RESC3216X70X50NL05T20
- RFB2, RFB3: footprint FP-ERJ3EK-MFG -> Vault:FP-ERJ3EK-MFG
- Rc1, Rc2: footprint RESC1005X40X25ML05T05 -> Vault:RESC1005X40X25ML05T05
- U10, U11: footprint DGK0008A_M -> Vault:DGK0008A_M
Changed lines of the file:
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@@
 		(in_pos_files yes)
 		(dnp no)
-		(property "Reference" "#PWR?"
+		(property "Reference" "#PWR011"
 			(at 104.14 104.14 0)
 			(hide yes)
@@
 			(project "LEARNSAT_POBOY_v3.2.0"
 				(path "/31302da5-a970-4b2b-aa05-afcd06cb9d09/0fb1b4e6-2835-46e5-a731-d5a5d61ae98c"
-					(reference "#PWR?")
+					(reference "#PWR011")
 					(unit 1)
 				)
@@
 			)
 		)
-		(property "Footprint" "FP-MLZ1608-IPC_C"
+		(property "Footprint" "Vault:FP-MLZ1608-IPC_C"
 			(at 63.5 124.46 0)
 			(hide yes)
@@
 			)
 		)
-		(property "Footprint" "FP-ERJ3EK-MFG"
+		(property "Footprint" "Vault:FP-ERJ3EK-MFG"
 			(at 119.38 66.04 0)
 			(hide yes)
@@
 			)
 		)
-		(property "Footprint" "RESC3216X70X50NL05T20"
+		(property "Footprint" "Vault:RESC3216X70X50NL05T20"
 			(at 127 142.24 0)
 			(hide yes)
@@
 		(in_pos_files yes)
 		(dnp no)
-		(property "Reference" "#PWR?"
+		(property "Reference" "#PWR010"
 			(at 68.58 190.5 0)
 			(hide yes)
@@
 			(project "LEARNSAT_POBOY_v3.2.0"
 				(path "/31302da5-a970-4b2b-aa05-afcd06cb9d09/0fb1b4e6-2835-46e5-a731-d5a5d61ae98c"
-					(reference "#PWR?")
+					(reference "#PWR010")
 					(unit 1)
 				)
@@
 		(in_pos_files yes)
 		(dnp no)
-		(property "Reference" "#PWR?"
+		(property "Reference" "#PWR08"
 			(at 55.88 190.5 0)
 			(hide yes)
@@
 			(project "LEARNSAT_POBOY_v3.2.0"
 				(path "/31302da5-a970-4b2b-aa05-afcd06cb9d09/0fb1b4e6-2835-46e5-a731-d5a5d61ae98c"
-					(reference "#PWR?")
+					(reference "#PWR08")
 					(unit 1)
 				)
@@
 		(in_pos_files yes)
 		(dnp no)
-		(property "Reference" "#PWR?"
+		(property "Reference" "#PWR016"
 			(at 124.46 190.5 0)
 			(hide yes)
@@
 			(project "LEARNSAT_POBOY_v3.2.0"
 				(path "/31302da5-a970-4b2b-aa05-afcd06cb9d09/0fb1b4e6-2835-46e5-a731-d5a5d61ae98c"
-					(reference "#PWR?")
+					(reference "#PWR016")
 					(unit 1)
 				)
@@
 			)
 		)
-		(property "Footprint" "DGK0008A_M"
+		(property "Footprint" "Vault:DGK0008A_M"
 			(at 78.74 50.8 0)
 			(hide yes)
@@
 			)
 		)
-		(property "Footprint" "FP-C0402-BB-MFG"
+		(property "Footprint" "Vault:FP-C0402-BB-MFG"
 			(at 63.5 91.44 0)
 			(hide yes)
@@
 			)
 		)
-		(property "Footprint" "FP-MLZ1608-IPC_C"
+		(property "Footprint" "Vault:FP-MLZ1608-IPC_C"
 			(at 58.42 38.1 0)
 			(hide yes)
@@
 		(in_pos_files yes)
 		(dnp no)
-		(property "Reference" "#PWR?"
+		(property "Reference" "#PWR017"
 			(at 134.62 104.14 0)
 			(hide yes)
@@
 			(project "LEARNSAT_POBOY_v3.2.0"
 				(path "/31302da5-a970-4b2b-aa05-afcd06cb9d09/0fb1b4e6-2835-46e5-a731-d5a5d61ae98c"
-					(reference "#PWR?")
+					(reference "#PWR017")
 					(unit 1)
 				)
@@
 			)
 		)
-		(property "Footprint" "DGK0008A_M"
+		(property "Footprint" "Vault:DGK0008A_M"
 			(at 83.82 137.16 0)
 			(hide yes)
@@
 		(in_pos_files yes)
 		(dnp no)
-		(property "Reference" "#PWR?"
+		(property "Reference" "#PWR012"
 			(at 109.22 190.5 0)
 			(hide yes)
@@
 			(project "LEARNSAT_POBOY_v3.2.0"
 				(path "/31302da5-a970-4b2b-aa05-afcd06cb9d09/0fb1b4e6-2835-46e5-a731-d5a5d61ae98c"
-					(reference "#PWR?")
+					(reference "#PWR012")
 					(unit 1)
 				)
@@
 		(in_pos_files yes)
 		(dnp no)
-		(property "Reference" "#PWR?"
+		(property "Reference" "#PWR014"
 			(at 116.84 190.5 0)
 			(hide yes)
@@
 			(project "LEARNSAT_POBOY_v3.2.0"
 				(path "/31302da5-a970-4b2b-aa05-afcd06cb9d09/0fb1b4e6-2835-46e5-a731-d5a5d61ae98c"
-					(reference "#PWR?")
+					(reference "#PWR014")
 					(unit 1)
 				)
@@
 			)
 		)
-		(property "Footprint" "FP-502-01-MFG"
+		(property "Footprint" "Vault:FP-502-01-MFG"
 			(at 99.06 124.46 0)
 			(hide yes)
@@
 		(in_pos_files yes)
 		(dnp no)
-		(property "Reference" "#PWR?"
+		(property "Reference" "#PWR07"
 			(at 50.8 104.14 0)
 			(hide yes)
@@
 			(project "LEARNSAT_POBOY_v3.2.0"
 				(path "/31302da5-a970-4b2b-aa05-afcd06cb9d09/0fb1b4e6-2835-46e5-a731-d5a5d61ae98c"
-					(reference "#PWR?")
+					(reference "#PWR07")
 					(unit 1)
 				)
@@
 			)
 		)
-		(property "Footprint" "RESC3216X70X50NL05T20"
+		(property "Footprint" "Vault:RESC3216X70X50NL05T20"
 			(at 121.92 55.88 0)
 			(hide yes)
@@
 		(in_pos_files yes)
 		(dnp no)
-		(property "Reference" "#PWR?"
+		(property "Reference" "#PWR015"
 			(at 119.38 104.14 0)
 			(hide yes)
@@
 			(project "LEARNSAT_POBOY_v3.2.0"
 				(path "/31302da5-a970-4b2b-aa05-afcd06cb9d09/0fb1b4e6-2835-46e5-a731-d5a5d61ae98c"
-					(reference "#PWR?")
+					(reference "#PWR015")
 					(unit 1)
 				)
@@
 			)
 		)
-		(property "Footprint" "FP-CL31-IPC_A"
+		(property "Footprint" "Vault:FP-CL31-IPC_A"
 			(at 50.8 73.66 0)
 			(hide yes)
@@
 			)
 		)
-		(property "Footprint" "FP-CL31-IPC_A"
+		(property "Footprint" "Vault:FP-CL31-IPC_A"
 			(at 134.62 68.58 0)
 			(hide yes)
@@
 			)
 		)
-		(property "Footprint" "RESC1005X40X25ML05T05"
+		(property "Footprint" "Vault:RESC1005X40X25ML05T05"
 			(at 71.12 162.56 0)
 			(hide yes)
@@
 			)
 		)
-		(property "Footprint" "FP-CL31-IPC_A"
+		(property "Footprint" "Vault:FP-CL31-IPC_A"
 			(at 139.7 154.94 0)
 			(hide yes)
@@
 		(in_pos_files yes)
 		(dnp no)
-		(property "Reference" "#PWR?"
+		(property "Reference" "#PWR09"
 			(at 63.5 104.14 0)
 			(hide yes)
@@
 			(project "LEARNSAT_POBOY_v3.2.0"
 				(path "/31302da5-a970-4b2b-aa05-afcd06cb9d09/0fb1b4e6-2835-46e5-a731-d5a5d61ae98c"
-					(reference "#PWR?")
+					(reference "#PWR09")
 					(unit 1)
 				)
@@
 			)
 		)
-		(property "Footprint" "FP-CL31-IPC_A"
+		(property "Footprint" "Vault:FP-CL31-IPC_A"
 			(at 55.88 160.02 0)
 			(hide yes)
@@
 		(in_pos_files yes)
 		(dnp no)
-		(property "Reference" "#PWR?"
+		(property "Reference" "#PWR018"
 			(at 139.7 190.5 0)
 			(hide yes)
@@
 			(project "LEARNSAT_POBOY_v3.2.0"
 				(path "/31302da5-a970-4b2b-aa05-afcd06cb9d09/0fb1b4e6-2835-46e5-a731-d5a5d61ae98c"
-					(reference "#PWR?")
+					(reference "#PWR018")
 					(unit 1)
 				)
@@
 			)
 		)
-		(property "Footprint" "FP-ERJ3EK-MFG"
+		(property "Footprint" "Vault:FP-ERJ3EK-MFG"
 			(at 124.46 152.4 0)
 			(hide yes)
@@
 		(in_pos_files yes)
 		(dnp no)
-		(property "Reference" "#PWR?"
+		(property "Reference" "#PWR013"
 			(at 111.76 104.14 0)
 			(hide yes)
@@
 			(project "LEARNSAT_POBOY_v3.2.0"
 				(path "/31302da5-a970-4b2b-aa05-afcd06cb9d09/0fb1b4e6-2835-46e5-a731-d5a5d61ae98c"
-					(reference "#PWR?")
+					(reference "#PWR013")
 					(unit 1)
 				)
@@
 			)
 		)
-		(property "Footprint" "FP-C0402-BB-MFG"
+		(property "Footprint" "Vault:FP-C0402-BB-MFG"
 			(at 68.58 177.8 0)
 			(hide yes)
@@
 			)
 		)
-		(property "Footprint" "FP-502-01-MFG"
+		(property "Footprint" "Vault:FP-502-01-MFG"
 			(at 93.98 38.1 0)
 			(hide yes)
@@
 			)
 		)
-		(property "Footprint" "RESC1005X40X25ML05T05"
+		(property "Footprint" "Vault:RESC1005X40X25ML05T05"
 			(at 66.04 76.2 0)
 			(hide yes)

Commit message: Edited 12V Rail schematics
Connections:
- net ??? renamed 12V
Changed lines of the file:
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@@
 		)
 	)
-	(global_label "???"
+	(global_label "12V"
 		(shape input)
 		(at 149.86 58.42 0)
@@
 		)
 		(property "Intersheetrefs" "${INTERSHEET_REFS}"
-			(at 156.111 58.42 0)
+			(at 156.3528 58.42 0)
 			(hide yes)
 			(show_name no)
@@
 		)
 	)
-	(global_label "???"
+	(global_label "12V"
 		(shape input)
 		(at 154.94 144.78 0)
@@
 		)
 		(property "Intersheetrefs" "${INTERSHEET_REFS}"
-			(at 161.191 144.78 0)
+			(at 161.4328 144.78 0)
 			(hide yes)
 			(show_name no)
