File: BoBa/BoBa.kicad_pcb (KiCad board)
At the start: 4 copper layers, 90.3 x 95.8 mm, 41 parts, among them J1 DF13C-2P-1.25V(21), J2 DF13C-2P-1.25V(21), J3 DF13C-2P-1.25V(21), J4 DF13C-2P-1.25V(21), Q1 FQD13N06LTM, Q2 FQD13N06LTM, U1 LTC4231HUD-2#TRPBF, U2 INA219, U3 INA219AIDCNR, U4_IN-A LTC4231IUD-2#TRPBF, U5 INA219AIDCNR

Commit message: Add files via upload
Routing:
- net INHIBIT: track 155.8 -> 163.2 mm
- net NetQ2_1: track 46.2 -> 50.0 mm
- net NetD1_1: track 74.9 -> 78.4 mm
- net 3V3_Secondary: track 155.3 -> 154.3 mm
- net NetQ2_4: track 72.2 -> 73.2 mm
- net NetR2_2: track 15.0 -> 15.8 mm
- net NetQ2_3: track 19.4 -> 20.0 mm

Commit message: Add files via upload
Parts:
- moved Q2 11.0 mm to (176.2, 79.9)
Routing:
- net Chassis GND: track 0.00 -> 153.3 mm
- net NetQ2_1: track 50.0 -> 68.9 mm
- net NetQ2_4: track 73.2 -> 87.8 mm
- net NetQ2_3: track 20.0 -> 28.3 mm
- net I2C Clock: track 107.8 -> 114.5 mm
- net 3V3_Secondary: track 154.3 -> 158.0 mm
- net NetD1_1: track 78.4 -> 82.0 mm
- net Vmppt: track 140.8 -> 143.4 mm
- net NetR2_2: track 15.8 -> 16.9 mm
- net Pack-_Neg: track 47.4 -> 48.0 mm
- net INHIBIT: track 163.2 -> 162.7 mm
- net I2C Data: track 100.9 -> 100.4 mm
